File: bluepill-industrial-shield.kicad_sch (KiCad schematic)
At the start: 11 parts, among them J1 Conn_01x02_Socket, J2 Conn_01x16_Socket, J3 Conn_01x02_Socket, J4 Conn_01x12_Socket, U1 BluePill, U2 TMA-2405D, U3 MAX3485

Commit message: trace pcb
Parts:
- added J4: Conn_01x02_Socket, Connector_Phoenix_MC:PhoenixContact_MCV_1,5_2-G-3.5_1x02_P3.50mm_Vertical, symbol Connector:Conn_01x02_Socket
- J5: renamed from J4; footprint Connector_Phoenix_MC:PhoenixContact_MCV_1,5_14-G-3.5_1x14_P3.50mm_Vertical -> Connector_Phoenix_MC:PhoenixContact_MCV_1,5_12-G-3.5_1x12_P3.50mm_Vertical; symbol Connector:Conn_01x14_Socket -> Connector:Conn_01x12_Socket
Connections:
- net OUT13 is gone; now on net IN13: U1.36 (PB8)
- net OUT14 is gone; now on net IN14: U1.37 (PB9)
- net +24V: now also J1.1 (Pin_1); no longer J1.2 (Pin_2)
- net GND: no longer J1.1 (Pin_1)
- net GND_IN: now also J1.2 (Pin_2)
- net IN10: now also U1.6 (PA1); no longer U1.7 (PA2)
- net IN11: now also U1.5 (PA0); no longer U1.6 (PA1)
- net IN12: now also U1.2 (PС13); no longer U1.5 (PA0)
- net IN13: no longer U1.4 (PС15)
- net IN14: no longer U1.3 (PС14)
- net IN5: now also U1.11 (PA6); no longer U1.12 (PA7)
- net IN6: now also U1.10 (PA5); no longer U1.11 (PA6)
- net IN7: now also U1.9 (PA4); no longer U1.10 (PA5)
- net IN8: now also U1.8 (PA3); no longer U1.9 (PA4)
- net IN9: now also U1.7 (PA2); no longer U1.8 (PA3)
- removed net DO13: J5.13 (Pin_13)
- removed net DO14: J5.14 (Pin_14)
- new net IP+: J4.1 (Pin_1)
- new net IP-: J4.2 (Pin_2)
- new net I_SENS: U1.12 (PA7)
- no-connect marks 4 -> 5
Other:
- sheet input ports: added IP+, IP-, I_SENS; removed none
- sheet output ports: added none; removed DO13, DO14, OUT13, OUT14
- moved on the sheet: J3

Commit message: add battery
Parts:
- added BT1: Battery_Cell, Battery:Battery_Panasonic_CR1220-VCN_Vertical_CircularHoles, symbol Device:Battery_Cell
Connections:
- net GND: now also BT1.2 (-)
- net +BATT: now reaches U1.1 (VBAT)
- net +BATT: now also BT1.1 (+)
- no-connect marks 5 -> 4

Commit message: update to kicad 9
Parts:
- H1, H2, H3, H4: footprint MountingHole:MountingHole_4.3mm_M4 -> MountingHole:MountingHole_3.2mm_M3
