File: input.kicad_sch (KiCad schematic)
At the start: 42 parts, among them U10 PC817, U11 PC817, U12 PC817, U13 PC817, U14 PC817, U15 PC817, U16 PC817, U17 PC817, U4 PC817, U5 PC817, U6 PC817, U7 PC817, U8 PC817, U9 PC817

Commit message: trace pcb
Parts:
- added C15: 100nF, Capacitor_SMD:C_0805_2012Metric, symbol Device:C
- added C16: 1nF, Capacitor_SMD:C_0805_2012Metric, symbol Device:C
- added C17: C, Capacitor_SMD:C_0805_2012Metric, symbol Device:C
- added R15, R17: 1K, Resistor_SMD:R_0805_2012Metric_Pad1.20x1.40mm_HandSolder, symbol Device:R
- added R16: 2K, Resistor_SMD:R_0805_2012Metric_Pad1.20x1.40mm_HandSolder, symbol Device:R
- added U18: ACS712xLCTR-05B, Package_SO:SOIC-8_3.9x4.9mm_P1.27mm, symbol Sensor_Current:ACS712xLCTR-05B
Connections:
- net GND: now also C15.2, C16.2, C17.2, R16.1, U18.5 (GND); no longer C1.2, C10.2, C11.2, C12.2, C13.2, C14.2, C2.2, C3.2, C4.2, C5.2, C6.2, C7.2, C8.2, C9.2, U10.2, U11.2, U12.2, U13.2, U14.2, U15.2, U16.2, U17.2, U4.2, U5.2, U6.2, U7.2, U8.2, U9.2
- new net: R15.1, U18.7 (VIOUT)
- new net: R15.2, R16.2, R17.1
- new net: C16.1, U18.6 (FILTER)
- new net +5V: C15.1, U18.8 (VCC)
- new net GND_IN: C1.2, C10.2, C11.2, C12.2, C13.2, C14.2, C2.2, C3.2, C4.2, C5.2, C6.2, C7.2, C8.2, C9.2, U10.2, U11.2, U12.2, U13.2, U14.2, U15.2, U16.2, U17.2, U4.2, U5.2, U6.2, U7.2, U8.2, U9.2
- new net IP+: U18.1 (IP+), U18.2 (IP+)
- new net IP-: U18.3 (IP-), U18.4 (IP-)
- new net I_SENS: C17.1, R17.2
